File: Leveltronic/Leveltronic.kicad_pcb (KiCad board)
At the start: 2 copper layers, 57 x 36 mm, 57 parts, among them J1 Header_100mil_1x06, J2 Header_100mil_1x02, J3 Header_100mil_1x02, J4 Header_100mil_1x02, U1 LMP7711MK, U2 LT1964ES5-SD, U3 TPS7A0218PDBVR, U4 LMP7711MK, U5 LMP7711MK

Commit message: Wylertronic basic board layout completed
Parts:
- added R14: 470R, sldrnrd:R_0805, F.Cu at (80.8, 52.4)
- R4, R5: value 1k -> 470R
- R7: value 10M -> 1M
- moved U5 44.6 mm to (69.4, 43.6), turned to -90 degrees
- moved R11 42.4 mm to (82.6, 44.8)
- moved C20 40.7 mm to (70.4, 48.8)
- moved C19 40.0 mm to (69.4, 38.4)
- moved C21 39.6 mm to (69.4, 40.4)
- moved R10 39.4 mm to (86.0, 44.8)
- moved C22 38.9 mm to (70.4, 46.8)
- moved U4 36.9 mm to (83.0, 47.8), turned to 180 degrees
- moved C15 34.3 mm to (88.2, 47.8), turned to -90 degrees
- moved C17 33.1 mm to (86.2, 47.8), turned to -90 degrees
- moved C16 27.9 mm to (77.8, 48.6), turned to -90 degrees
- moved C18 27.4 mm to (79.8, 48.6), turned to -90 degrees
- moved C23 27.0 mm to (76.0, 44.8), turned to 180 degrees
- moved J2 19.5 mm to (77.1, 52.5), turned to -90 degrees
- moved R7 19.1 mm to (88.0, 51.4), turned to -90 degrees
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Connections:
- R1 pad 1: Pendulum -> Net-(U1-+IN)
- U1 pad 3: Pendulum -> Net-(U1-+IN)
- U4 pad 3: Pendulum -> Net-(U1-+IN)
Routing:
- net 1V8: track 0.00 -> 68.6 mm, vias 0 -> 4
- net Output: track 0.00 -> 63.7 mm
- net -1V8: track 0.00 -> 52.8 mm
- net ExciterA: track 0.00 -> 45.8 mm
- net ExciterB: track 0.00 -> 38.0 mm
- net Net-(D1-K): track 0.00 -> 36.4 mm
- net Net-(RV1-Wiper): track 0.00 -> 35.0 mm
- net Net-(D3-A): track 0.00 -> 19.6 mm
- net PendulumShield: track 0.00 -> 18.1 mm
- net Net-(RV2-Wiper): track 0.00 -> 15.9 mm
- net Net-(RV2-CW): track 0.00 -> 10.4 mm
- net Net-(RV1-CW): track 0.00 -> 9.68 mm
- net Net-(U1-+IN): track 0.00 -> 8.85 mm
- net Net-(U4-OUT): track 0.00 -> 6.75 mm
- net Net-(U4--IN): track 0.00 -> 6.28 mm
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Other:
- board text added: "Gain"
- board text added: "Zero"
