File: Leveltronic/Leveltronic.kicad_pcb (KiCad board)
At the start: 2 copper layers, 57 x 36 mm, 61 parts, among them J1 Header_100mil_1x06, J2 Header_100mil_1x04, J3 Header_100mil_1x02, J4 Header_100mil_1x02, J5 Header_100mil_1x02, U1 LMP7711MK, U2 LT1964ES5-SD, U3 LDK130M18R, U4 LMP7711MK, U5 LMP7711MK

Commit message: Leveltronic board fully layed out
Parts:
- added J6: Header_50mil_1x02, sldrnrd:Header_50mil_1x02, F.Cu at (78.4, 55.0)
- J2: value Header_100mil_1x04 -> Header_100mil_1x03; footprint sldrnrd:Header_100mil_1x04 -> sldrnrd:Header_100mil_1x03
- J3, J4: value Header_100mil_1x02 -> Header_50mil_1x02; footprint sldrnrd:Header_100mil_1x02 -> sldrnrd:Header_50mil_1x02
- moved J3 33.3 mm to (69.2, 64.2), turned to -90 degrees
- moved J4 25.5 mm to (72.0, 64.2), turned to -90 degrees
- moved C5 4.08 mm to (56.4, 49.3)
- moved C6 4.08 mm to (58.6, 50.5)
- moved C7 4.08 mm to (67.2, 49.5)
- moved R6 4.08 mm to (60.8, 47.7)
- moved R8 4.08 mm to (64.2, 47.7)
- moved U2 4.08 mm to (61.8, 50.5)
- moved C8 4.08 mm to (65.0, 50.7)
- moved RV2 3.40 mm to (80.5, 42.0)
- moved J1 3.35 mm to (44.2, 53.0), turned to -90 degrees
- moved C1 3.27 mm to (56.2, 57.7)
- moved C3 3.27 mm to (67.0, 57.9)
- moved D3 3.27 mm to (52.5, 52.9)
- moved D4 3.27 mm to (52.5, 57.9)
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Connections:
- J1 pad 1: Output -> GND
- J1 pad 2: ExciterB -> 5V0
- J1 pad 3: ExciterA -> -5V0
- J1 pad 4: GND -> ExciterA
- J1 pad 5: -5V0 -> ExciterB
- J1 pad 6: 5V0 -> Output
- J2 pad 1: Pendulum -> GND
- J2 pad 3: PendulumShield -> Pendulum
- J5 pad 1: Net-(U4-OUT) -> GND
- J5 pad 2: GND -> Net-(U4-OUT)
Routing:
- net -1V8: track 51.4 -> 46.9 mm
- net Pendulum: track 2.81 -> 7.06 mm
- net PendulumShield: track 18.1 -> 21.3 mm
- net Net-(RV2-Wiper): track 15.9 -> 13.1 mm
- net ExciterA: track 45.8 -> 43.1 mm
- net 5V0: track 2.82 -> 5.22 mm
- net -5V0: track 2.80 -> 5.11 mm
- net Net-(RV1-Wiper): track 47.4 -> 49.4 mm
- net Net-(D3-A): track 19.6 -> 21.5 mm
- net 1V8: track 70.8 -> 69.5 mm, vias 4 -> 2
- net Net-(RV2-CCW): track 3.65 -> 4.81 mm
- net Output: track 63.7 -> 63.0 mm
- net GND: track 0.00 -> 0.35 mm, vias 0 -> 65
- added copper zone on B.Cu, net GND
- added copper zone on F.Cu, net GND
Other:
- board text added: "+5V"
- board text added: "-5V"
- board text added: "A"
- board text added: "B"
- board text added: "GND"
- board text added: "Out"
- board text added: "soldernerd"
- board text added: "soldernerd.com LEVELTRONIC 2026 - Rev A"
