File: Leveltronic/Leveltronic-hexacore.kicad_pcb (KiCad board)
At the start: 2 copper layers, 57 x 36 mm, 61 parts, among them J1 Header_100mil_1x06, J2 Header_100mil_1x04, J3 Header_100mil_1x02, J4 Header_100mil_1x02, J5 Header_100mil_1x02, U1 LMP7711MK, U2 LT1964ES5-SD, U3 LDK130M18R, U4 LMP7711MK, U5 LMP7711MK

Commit message: Some universality added, positive LDO replaced
Parts:
- removed C9: 10n, sldrnrd:C_0805
- removed J5: Header_100mil_1x02, sldrnrd:Header_100mil_1x02
- removed R17: Opt, sldrnrd:R_0805
- J2: value Header_100mil_1x04 -> Header_100mil_1x02; footprint sldrnrd:Header_100mil_1x04 -> sldrnrd:Header_100mil_1x02
- R14: value 470R -> 100R
- R4, R5: value 470R -> 1k
- R7: value 1M -> 10M
- U3: value LDK130M18R -> TPS7A0218PDBVR
- moved R7 19.1 mm to (74.2, 64.6), turned to 0 degrees
- moved R9 15.5 mm to (74.0, 62.2), turned to 0 degrees
- moved R15 13.2 mm to (67.6, 46.8), turned to -90 degrees
- moved R1 13.0 mm to (74.0, 60.0)
- moved R16 11.5 mm to (86.6, 43.0), turned to 0 degrees
- moved R12 11.3 mm to (85.6, 62.4), turned to 90 degrees
- moved R6 10.1 mm to (66.8, 53.8), turned to 0 degrees
- moved R13 8.12 mm to (80.2, 62.4), turned to -90 degrees
- moved R8 6.55 mm to (67.2, 51.4), turned to 0 degrees
- moved R10 5.69 mm to (82.4, 49.2)
- moved R14 4.07 mm to (79.3, 48.6)
- moved C13 3.74 mm to (73.8, 55.4)
- moved C14 3.74 mm to (71.8, 55.4)
- moved C11 3.74 mm to (82.4, 54.6)
- moved C12 3.74 mm to (80.4, 54.6)
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Connections:
- U3 pad 4: Net-(U3-BYP) -> unconnected-(U3-N/C-Pad4)
Routing:
- net 1V8: track 70.8 -> 0.00 mm, vias 4 -> 0
- net Output: track 63.7 -> 0.00 mm
- net -1V8: track 51.4 -> 0.00 mm
- net Net-(RV1-Wiper): track 47.4 -> 0.00 mm
- net ExciterA: track 45.8 -> 0.00 mm
- net ExciterB: track 38.0 -> 0.00 mm
- net Net-(D1-K): track 36.4 -> 0.00 mm
- net Net-(D3-A): track 19.6 -> 0.00 mm
- net PendulumShield: track 18.1 -> 0.00 mm
- net Net-(RV2-Wiper): track 15.9 -> 0.00 mm
- net Net-(U4-OUT): track 12.3 -> 0.00 mm
- net Net-(RV2-CW): track 10.4 -> 0.00 mm
- net Net-(RV1-CW): track 9.68 -> 0.00 mm
- net Net-(U1-+IN): track 8.85 -> 0.00 mm
- net Net-(R1-Pad2): track 6.97 -> 0.00 mm
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Other:
- board text removed: "Gain"
- board text removed: "Zero"
