File: Leveltronic/Leveltronic.kicad_sch (KiCad schematic)
At the start: 57 parts, among them J1 Header_100mil_1x06, J2 Header_100mil_1x02, J3 Header_100mil_1x02, J4 Header_100mil_1x02, U1 LMP7711MK, U2 LT1964ES5-SD, U3 TPS7A0218PDBVR, U4 LMP7711MK, U5 LMP7711MK

Commit message: Wylertronic basic board layout completed
Parts:
- added R14: 470R, sldrnrd:R_0805, symbol sldrnrd:Resistor/R0805_470R
- R4, R5: value 1k -> 470R; symbol sldrnrd:Resistor/R0805_1k -> sldrnrd:Resistor/R0805_470R; LCSC C17513 -> C17710; MPN 0805W8F1001T5E -> 0805W8F4700T5E
- R7: value 10M -> 1M; symbol sldrnrd:Resistor/R0805_10M -> sldrnrd:Resistor/R0805_1M; LCSC C325772 -> C17514; MPN 0805W8F1005T5E -> 0805W8F1004T5E
Connections:
- net Pendulum: now also R14.1; no longer R1.1, U1.3 (+IN), U4.3 (+IN)
- new net: R1.1, R14.2, U1.3 (+IN), U4.3 (+IN)
Other:
- moved on the sheet: C11, C12, C15, C16, C17, C18, C20, C22, R10, R11

Commit message: Some universality added, positive LDO replaced
Parts:
- added C9: 10n, sldrnrd:C_0805, symbol sldrnrd:Capacitor/C0805_10n
- added J5: Header_100mil_1x02, sldrnrd:Header_100mil_1x02, symbol sldrnrd:Connector/100Mil/Header_100mil_1x02
- added R17: Opt, sldrnrd:R_0805, symbol sldrnrd:Resistor/R0805_10M
- J2: value Header_100mil_1x02 -> Header_100mil_1x04; footprint sldrnrd:Header_100mil_1x02 -> sldrnrd:Header_100mil_1x04; symbol sldrnrd:Connector/100Mil/Header_100mil_1x02 -> sldrnrd:Connector/100Mil/Header_100mil_1x04; LCSC C225477 -> C225479; MPN A2541WV-2P -> A2541WV-4P
- U3: value TPS7A0218PDBVR -> LDK130M18R; symbol sldrnrd:Power/LinearRegulator/TPS7A0218PDBVR -> sldrnrd:Power/LinearRegulator/LDK130M18R; LCSC C3748843 -> C377955; MPN TPS7A0218PDBVR -> LDK130M18R; Manufacturer Texas Instruments -> STMicroelectronics
Connections:
- net GND: now also J2.4, C9.2, J5.2; no longer C11.2, C12.2
- net PendulumShield: now also J2.3
- net at C23.2, RV1.2 (Wiper), U5.3 (+IN): now also R17.2
- net at R1.2, R7.2, R9.2: now also R17.1
- net at C23.1, R11.1, U4.1 (OUT): now also J5.1
- net at U3.4 (BYP): now also C9.1

Commit message: Leveltronic board fully layed out
Parts:
- added J6: Header_50mil_1x02, sldrnrd:Header_50mil_1x02, symbol sldrnrd:Connector/50Mil/Header_50mil_1x02
- J2: value Header_100mil_1x04 -> Header_100mil_1x03; footprint sldrnrd:Header_100mil_1x04 -> sldrnrd:Header_100mil_1x03; symbol sldrnrd:Connector/100Mil/Header_100mil_1x04 -> sldrnrd:Connector/100Mil/Header_100mil_1x03; LCSC C225479 -> C225478; MPN A2541WV-4P -> A2541WV-3P
- J3, J4: value Header_100mil_1x02 -> Header_50mil_1x02; footprint sldrnrd:Header_100mil_1x02 -> sldrnrd:Header_50mil_1x02; symbol sldrnrd:Connector/100Mil/Header_100mil_1x02 -> sldrnrd:Connector/50Mil/Header_50mil_1x02
Connections:
- net -5V0: now also J1.3; no longer J1.5
- net 5V0: now also J1.2; no longer J1.6
- net ExciterA: now also J1.4, J3.02 (2); no longer J1.3, J3.1
- net ExciterB: now also J1.5, J4.02 (2); no longer J1.2, J4.1
- net GND: now also C11.2, C12.2, J1.1, J2.1, J3.01 (1), J4.01 (1), J5.1; no longer J1.4, J2.4, J3.2, J4.2, J5.2
- net Output: now also J1.6; no longer J1.1
- net Pendulum: now also J2.3, J6.02 (2); no longer J2.1
- net PendulumShield: now also J6.01 (1); no longer J2.3
- net at C23.1, R11.1, U4.1 (OUT): now also J5.2; no longer J5.1
Other:
- moved on the sheet: J3, J4
