File: mcu.kicad_sch (KiCad schematic)
At the start: 12 parts, among them U6 STM32G0B1RET6, U7 RN4871-I/RM128, Y1 Q13FC1350000400, Y2 X50328MSB2GI

Commit message: Schematic and component placement semi-final. Routing pending
Connections:
- net BLE_P1_6: no longer U6.3 (PC13)
- net BLE_P1_7: no longer U6.59 (PB5)
- net BLE_P2_0: no longer U6.1 (PC11)
- net BLE_P3_6: no longer U6.64 (PC10)
- net ~{BLE_RST}: now also U6.59 (PB5); no longer U6.2 (PC12)
- net ADC_CLOCK: now reaches U6.30 (PB10)
- net PCAP04_1_INT: no longer names the net of U6.37 (PA9)
- net PCAP04_1_P2: no longer names the net of U6.36 (PA8)
- net PCAP04_1_P3: no longer names the net of U6.35 (PB15)
- net PCAP04_1_SCL: no longer names the net of U6.33 (PB13)
- net PCAP04_1_SDA: no longer names the net of U6.34 (PB14)
- net PCAP04_2_INT renamed ADC_READY
- net PCAP04_2_P2 renamed ADC_SYNC_RESET
- net PCAP04_2_P3: no longer names the net of U6.15 (PC2)
- net PCAP04_2_SCL: no longer names the net of U6.13 (PC0)
- net PCAP04_2_SDA: no longer names the net of U6.14 (PC1)
- net SCL3300_CS renamed ADC_CS
- net SCL3300_MISO renamed ADC_MISO
- net SCL3300_MOSI renamed ADC_MOSI
- net SCL3300_SCK renamed ADC_SCK
- new net DAC_Clock: U6.1 (PC11)
- new net DAC_FSYNC: U6.3 (PC13)
- new net DAC_MOSI: U6.2 (PC12)
- new net DAC_SCK: U6.64 (PC10)
Other:
- note added: "SPI3"
- note added: "TMR1_CH4"
- note added: "TMR2_CH3"
- note added: "TMR3_CH4"
- note removed: "I2C2"

Commit message: Board layout without errors
Parts:
- renumbered C16 to C22, C17 to C23, C18 to C24, C19 to C25, C20 to C26, C21 to C27, C22 to C28, C23 to C29, U6 to U7, U7 to U8
Changed lines of the file:
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@@
 		(in_pos_files yes)
 		(dnp no)
-		(property "Reference" "#PWR43"
+		(property "Reference" "#PWR055"
 			(at 62.23 185.42 0)
 			(hide yes)
@@
 			(project "Levelmeter"
 				(path "/7d35597c-fbf9-4ce7-8410-0e7922679ea3/c7060150-8e88-4322-90f4-a2380d2eedad"
-					(reference "#PWR43")
+					(reference "#PWR055")
 					(unit 1)
 				)
@@
 		(in_pos_files yes)
 		(dnp no)
-		(property "Reference" "U7"
+		(property "Reference" "U8"
 			(at 315.976 131.064 0)
 			(show_name no)
@@
 			(project "Levelmeter"
 				(path "/7d35597c-fbf9-4ce7-8410-0e7922679ea3/c7060150-8e88-4322-90f4-a2380d2eedad"
-					(reference "U7")
+					(reference "U8")
 					(unit 1)
 				)
@@
 		(in_pos_files yes)
 		(dnp no)
-		(property "Reference" "#PWR44"
+		(property "Reference" "#PWR056"
 			(at 71.12 185.42 0)
 			(hide yes)
@@
 			(project "Levelmeter"
 				(path "/7d35597c-fbf9-4ce7-8410-0e7922679ea3/c7060150-8e88-4322-90f4-a2380d2eedad"
-					(reference "#PWR44")
+					(reference "#PWR056")
 					(unit 1)
 				)
@@
 		(in_pos_files yes)
 		(dnp no)
-		(property "Reference" "#PWR48"
+		(property "Reference" "#PWR060"
 			(at 361.95 161.29 0)
 			(hide yes)
@@
 			(project "Levelmeter"
 				(path "/7d35597c-fbf9-4ce7-8410-0e7922679ea3/c7060150-8e88-4322-90f4-a2380d2eedad"
-					(reference "#PWR48")
+					(reference "#PWR060")
 					(unit 1)
 				)
@@
 		(dnp no)
 		(fields_autoplaced yes)
-		(property "Reference" "#PWR42"
+		(property "Reference" "#PWR054"
 			(at 62.23 80.01 0)
 			(hide yes)
@@
 			(project "Levelmeter"
 				(path "/7d35597c-fbf9-4ce7-8410-0e7922679ea3/c7060150-8e88-4322-90f4-a2380d2eedad"
-					(reference "#PWR42")
+					(reference "#PWR054")
 					(unit 1)
 				)
@@
 		(in_pos_files yes)
 		(dnp no)
-		(property "Reference" "C22"
+		(property "Reference" "C28"
 			(at 88.9 142.24 90)
 			(show_name no)
@@
 			(project "Levelmeter"
 				(path "/7d35597c-fbf9-4ce7-8410-0e7922679ea3/c7060150-8e88-4322-90f4-a2380d2eedad"
-					(reference "C22")
+					(reference "C28")
 					(unit 1)
 				)
@@
 		(in_pos_files yes)
 		(dnp no)
-		(property "Reference" "#PWR45"
+		(property "Reference" "#PWR057"
 			(at 81.28 185.42 0)
 			(hide yes)
@@
 			(project "Levelmeter"
 				(path "/7d35597c-fbf9-4ce7-8410-0e7922679ea3/c7060150-8e88-4322-90f4-a2380d2eedad"
-					(reference "#PWR45")
+					(reference "#PWR057")
 					(unit 1)
 				)
@@
 		(in_pos_files yes)
 		(dnp no)
-		(property "Reference" "#PWR47"
+		(property "Reference" "#PWR059"
 			(at 295.91 161.29 0)
 			(hide yes)
@@
 			(project "Levelmeter"
 				(path "/7d35597c-fbf9-4ce7-8410-0e7922679ea3/c7060150-8e88-4322-90f4-a2380d2eedad"
-					(reference "#PWR47")
+					(reference "#PWR059")
 					(unit 1)
 				)
@@
 		(in_pos_files yes)
 		(dnp no)
-		(property "Reference" "C19"
+		(property "Reference" "C25"
 			(at 88.9 109.22 90)
 			(show_name no)
@@
 			(project "Levelmeter"
 				(path "/7d35597c-fbf9-4ce7-8410-0e7922679ea3/c7060150-8e88-4322-90f4-a2380d2eedad"
-					(reference "C19")
+					(reference "C25")
 					(unit 1)
 				)
@@
 		(in_pos_files yes)
 		(dnp no)
-		(property "Reference" "U6"
+		(property "Reference" "U7"
 			(at 159.258 127 0)
 			(show_name no)
@@
 			(project "Levelmeter"
 				(path "/7d35597c-fbf9-4ce7-8410-0e7922679ea3/c7060150-8e88-4322-90f4-a2380d2eedad"
-					(reference "U6")
+					(reference "U7")
 					(unit 1)
 				)
@@
 		(in_pos_files yes)
 		(dnp no)
-		(property "Reference" "#PWR49"
+		(property "Reference" "#PWR061"
 			(at 373.38 115.57 0)
 			(hide yes)
@@
 			(project "Levelmeter"
 				(path "/7d35597c-fbf9-4ce7-8410-0e7922679ea3/c7060150-8e88-4322-90f4-a2380d2eedad"
-					(reference "#PWR49")
+					(reference "#PWR061")
 					(unit 1)
 				)
@@
 		(in_pos_files yes)
 		(dnp no)
-		(property "Reference" "C20"
+		(property "Reference" "C26"
 			(at 88.9 119.38 90)
 			(show_name no)
@@
 			(project "Levelmeter"
 				(path "/7d35597c-fbf9-4ce7-8410-0e7922679ea3/c7060150-8e88-4322-90f4-a2380d2eedad"
-					(reference "C20")
+					(reference "C26")
 					(unit 1)
 				)
@@
 		(in_pos_files yes)
 		(dnp no)
-		(property "Reference" "C18"
+		(property "Reference" "C24"
 			(at 73.66 133.35 90)
 			(show_name no)
@@
 			(project "Levelmeter"
 				(path "/7d35597c-fbf9-4ce7-8410-0e7922679ea3/c7060150-8e88-4322-90f4-a2380d2eedad"
-					(reference "C18")
+					(reference "C24")
 					(unit 1)
 				)
@@
 		(in_pos_files yes)
 		(dnp no)
-		(property "Reference" "C23"
+		(property "Reference" "C29"
 			(at 375.92 143.51 90)
 			(show_name no)
@@
 			(project "Levelmeter"
 				(path "/7d35597c-fbf9-4ce7-8410-0e7922679ea3/c7060150-8e88-4322-90f4-a2380d2eedad"
-					(reference "C23")
+					(reference "C29")
 					(unit 1)
 				)
@@
 		(in_pos_files yes)
 		(dnp no)
-		(property "Reference" "#PWR41"
+		(property "Reference" "#PWR053"
 			(at 52.07 185.42 0)
 			(hide yes)
@@
 			(project "Levelmeter"
 				(path "/7d35597c-fbf9-4ce7-8410-0e7922679ea3/c7060150-8e88-4322-90f4-a2380d2eedad"
-					(reference "#PWR41")
+					(reference "#PWR053")
 					(unit 1)
 				)
@@
 		(in_pos_files yes)
 		(dnp no)
-		(property "Reference" "C21"
+		(property "Reference" "C27"
 			(at 88.9 132.08 90)
 			(show_name no)
@@
 			(project "Levelmeter"
 				(path "/7d35597c-fbf9-4ce7-8410-0e7922679ea3/c7060150-8e88-4322-90f4-a2380d2eedad"
-					(reference "C21")
+					(reference "C27")
 					(unit 1)
 				)
@@
 		(in_pos_files yes)
 		(dnp no)
-		(property "Reference" "#PWR50"
+		(property "Reference" "#PWR062"
 			(at 373.38 161.29 0)
 			(hide yes)
@@
 			(project "Levelmeter"
 				(path "/7d35597c-fbf9-4ce7-8410-0e7922679ea3/c7060150-8e88-4322-90f4-a2380d2eedad"
-					(reference "#PWR50")
+					(reference "#PWR062")
 					(unit 1)
 				)
@@
 		(in_pos_files yes)
 		(dnp no)
-		(property "Reference" "C16"
+		(property "Reference" "C22"
 			(at 54.61 133.35 90)
 			(show_name no)
@@
 			(project "Levelmeter"
 				(path "/7d35597c-fbf9-4ce7-8410-0e7922679ea3/c7060150-8e88-4322-90f4-a2380d2eedad"
-					(reference "C16")
+					(reference "C22")
 					(unit 1)
 				)
@@
 		(in_pos_files yes)
 		(dnp no)
-		(property "Reference" "C17"
+		(property "Reference" "C23"
 			(at 64.77 133.35 90)
 			(show_name no)
@@
 			(project "Levelmeter"
 				(path "/7d35597c-fbf9-4ce7-8410-0e7922679ea3/c7060150-8e88-4322-90f4-a2380d2eedad"
-					(reference "C17")
+					(reference "C23")
 					(unit 1)
 				)
@@
 		(in_pos_files yes)
 		(dnp no)
-		(property "Reference" "#PWR46"
+		(property "Reference" "#PWR058"
 			(at 116.84 185.42 0)
 			(hide yes)
@@
 			(project "Levelmeter"
 				(path "/7d35597c-fbf9-4ce7-8410-0e7922679ea3/c7060150-8e88-4322-90f4-a2380d2eedad"
-					(reference "#PWR46")
+					(reference "#PWR058")
 					(unit 1)
 				)

Commit message: BLE module: footprint fixed (keepout areas), additional pins routed to MCU, 3-pin 50mil debug header added
Parts:
- added J8: Header_100mil_1x02, sldrnrd:Header_50mil_1x03, symbol sldrnrd:Connector/50Mil/Header_50mil_1x03
- C29: value 100n -> 10u; footprint sldrnrd:C_0603 -> sldrnrd:C_1206; symbol sldrnrd:Capacitor/C0603_100n -> sldrnrd:Capacitor/C1206_10u; LCSC C14663 -> C70462; MPN CC0603KRX7R9BB104 -> CC1206KKX7R8BB106; Voltage 50V -> 25V
Connections:
- net BLE_P0_2: no longer U7.58 (PB4)
- net BLE_P1_6: now also U7.37 (PA9)
- net BLE_P1_7: now also U7.36 (PA8)
- net BLE_UART_BLE_TO_MCU: now also J8.03 (3)
- net BLE_UART_MCU_TO_BLE: now also J8.02 (2)
- net GND: now also J8.01 (1)
- net BLE_P0_0: now reaches U8.11 (P0_0)
- net BLE_P2_7: now reaches U8.15 (P2_7)
- net BLE_P1_2: now reaches U8.3 (P1_2)
- net BLE_P1_2: now also U7.58 (PB4)
- net BLE_P1_3: now reaches U8.4 (P1_3)
- net BLE_P1_3: now also U7.35 (PB15)

Commit message: Debug headers for SPI1, SPI2 and SPI3 added
Parts:
- J8: value Header_100mil_1x02 -> Header_50mil_1x03
Changed lines of the file:
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@@
 	(text "SPI3"
 		(exclude_from_sim no)
-		(at 108.712 90.17 0)
+		(at 113.284 93.218 0)
 		(effects
 			(font
@@
 		(in_pos_files yes)
 		(dnp no)
-		(fields_autoplaced yes)
 		(property "Reference" "J8"
 			(at 313.69 173.9899 0)
@@
 					(size 1.27 1.27)
 				)
-				(justify left)
-			)
-		)
-		(property "Value" "Header_100mil_1x02"
-			(at 313.69 176.5299 0)
-			(show_name no)
-			(do_not_autoplace no)
-			(effects
-				(font
-					(size 1.27 1.27)
-				)
-				(justify left)
-			)
-		)
+			)
+		)
+		(property "Value" "Header_50mil_1x03"
+			(at 310.134 180.848 0)
+			(show_name no)
+			(do_not_autoplace no)
+			(effects
+				(font
+					(size 1.27 1.27)
+				)
+			)
+		)

Commit message: Pinout description added, STM configuration added, netlist exported
Connections:
- net ~{CHARGE_EN} renamed CHARGE_EN
Changed lines of the file:
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@@
 		)
 	)
-	(global_label "~{CHARGE_EN}"
+	(global_label "CHARGE_EN"
 		(shape output)
 		(at 162.56 82.55 90)

Commit message: Schematic checks, some smaller corrections, debug UART pinout corrected on programming header
Connections:
- net CHARGE_EN renamed ~{CHARGE_EN}
Changed lines of the file:
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@@
 		)
 	)
-	(global_label "CHARGE_EN"
+	(global_label "~{CHARGE_EN}"
 		(shape output)
 		(at 162.56 82.55 90)
@@
 		)
 	)
-	(embedded_fonts no)
 )

Commit message: Further checks. Capacitors unified to basic parts
Parts:
- C29: footprint sldrnrd:C_1206 -> sldrnrd:C_0805; symbol sldrnrd:Capacitor/C1206_10u -> sldrnrd:Capacitor/C0805_10u; Dielectric X7R -> X5R; LCSC C70462 -> C440198; MPN CC1206KKX7R8BB106 -> GRM21BR61H106KE43L; Manufacturer Yageo -> Murata; Voltage 25V -> 50V
Changed lines of the file:
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@@
 	)
 	(symbol
-		(lib_id "sldrnrd:Capacitor/C1206_10u")
+		(lib_id "sldrnrd:Capacitor/C0805_10u")
 		(at 373.38 143.51 0)
 		(unit 1)
@@
 			)
 		)
-		(property "Footprint" "sldrnrd:C_1206"
+		(property "Footprint" "sldrnrd:C_0805"
 			(at 373.38 143.51 0)
 			(hide yes)
@@
 			)
 		)
-		(property "Description" "10uF Capacitor, 1206"
+		(property "Description" "10uF Capacitor, 0805"
 			(at 373.38 143.51 0)
 			(hide yes)
@@
 			)
 		)
-		(property "LCSC" "C70462"
+		(property "LCSC" "C440198"
 			(at 373.38 143.51 0)
 			(hide yes)
@@
 			)
 		)
-		(property "Dielectric" "X7R"
+		(property "Dielectric" "X5R"
 			(at 373.38 143.51 0)
 			(hide yes)
@@
 			)
 		)
-		(property "Voltage" "25V"
+		(property "Voltage" "50V"
 			(at 373.38 143.51 0)
 			(hide yes)
@@
 			)
 		)
-		(property "Manufacturer" "Yageo"
+		(property "Manufacturer" "Murata"
 			(at 373.38 143.51 0)
 			(hide yes)
@@
 			)
 		)
-		(property "MPN" "CC1206KKX7R8BB106"
+		(property "MPN" "GRM21BR61H106KE43L"
 			(at 373.38 143.51 0)
 			(hide yes)
@@
 		)
 	)
+	(embedded_fonts no)
 )

Commit message: LEVELMETER Rev A as ordered
Parts:
- added R58, R59: 22R, sldrnrd:R_0603, symbol sldrnrd:Resistor/R0603_22R
Connections:
- net ADC_CLOCK: now also R59.1; no longer U7.30 (PB10)
- net DAC_Clock: now also R58.1; no longer U7.1 (PC11)
- new net: R59.2, U7.30 (PB10)
- new net: R58.2, U7.1 (PC11)
