File: mcu.kicad_sch (KiCad schematic)
At the start: 15 parts, among them J8 Header_50mil_1x03, U7 STM32G0B1RET6, U8 RN4871-I/RM128, Y1 Q13FC1350000400, Y2 X50328MSB2GI

Commit message: Revision B semi-final
Connections:
- net I2C3_SCL: now reaches U7.13 (PC0)
- net I2C3_SDA: now reaches U7.14 (PC1)
- net SPI1_CS2: now reaches U7.42 (PA10)
- net AUX1: now reaches U7.47 (PA15)
- net AUX2: now reaches U7.48 (PC8)
Changed lines of the file:
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@@
 	(wire
 		(pts
+			(xy 113.03 143.51) (xy 120.65 143.51)
+		)
+		(stroke
+			(width 0)
+			(type default)
+		)
+	)
+	(wire
+		(pts
 			(xy 331.47 118.11) (xy 340.36 118.11)
 		)
@@
 	(wire
 		(pts
+			(xy 113.03 147.32) (xy 120.65 147.32)
+		)
+		(stroke
+			(width 0)
+			(type default)
+		)
+	)
+	(wire
+		(pts
 			(xy 135.89 82.55) (xy 135.89 86.36)
 		)
@@
 	(wire
 		(pts
+			(xy 200.66 97.79) (xy 205.74 97.79)
+		)
+		(stroke
+			(width 0)
+			(type default)
+		)
+	)
+	(wire
+		(pts
 			(xy 302.26 172.72) (xy 298.45 172.72)
 		)
@@
 	(wire
 		(pts
+			(xy 200.66 120.65) (xy 205.74 120.65)
+		)
+		(stroke
+			(width 0)
+			(type default)
+		)
+	)
+	(wire
+		(pts
 			(xy 331.47 133.35) (xy 340.36 133.35)
 		)
@@
 	(wire
 		(pts
+			(xy 200.66 101.6) (xy 205.74 101.6)
+		)
+		(stroke
+			(width 0)
+			(type default)
+		)
+	)
+	(wire
+		(pts
 			(xy 300.99 175.26) (xy 300.99 173.99)
 		)
@@
 		)
 	)
+	(global_label "AUX1"
+		(shape bidirectional)
+		(at 205.74 101.6 0)
+		(fields_autoplaced yes)
+		(effects
+			(font
+				(size 1.27 1.27)
+			)
+			(justify left)
+		)
+		(property "Intersheetrefs" "${INTERSHEET_REFS}"
+			(at 214.6746 101.6 0)
+			(show_name no)
+			(do_not_autoplace no)
+			(effects
+				(font
+					(size 1.27 1.27)
+				)
+				(justify left)
+			)
+		)
+	)
 	(global_label "DISP_ON"
 		(shape output)
@@
 		)
 	)
+	(global_label "I2C3_SCL"
+		(shape bidirectional)
+		(at 113.03 143.51 180)
+		(effects
+			(font
+				(size 1.27 1.27)
+			)
+			(justify right)
+		)
+		(property "Intersheetrefs" "${INTERSHEET_REFS}"
+			(at 113.03 143.51 0)
+			(show_name no)
+			(do_not_autoplace no)
+			(effects
+				(font
+					(size 1.27 1.27)
+				)
+			)
+		)
+		(property "Intersheetref" "${INTERSHEET_REFS}"
+			(at 113.03 143.51 0)
+			(hide yes)
+			(show_name no)
+			(do_not_autoplace no)
+			(effects
+				(font
+					(size 1.27 1.27)
+				)
+			)
+		)
+	)
 	(global_label "SWDIO"
 		(shape bidirectional)
@@
 		)
 	)
+	(global_label "AUX2"
+		(shape bidirectional)
+		(at 205.74 97.79 0)
+		(fields_autoplaced yes)
+		(effects
+			(font
+				(size 1.27 1.27)
+			)
+			(justify left)
+		)
+		(property "Intersheetrefs" "${INTERSHEET_REFS}"
+			(at 214.6746 97.79 0)
+			(show_name no)
+			(do_not_autoplace no)
+			(effects
+				(font
+					(size 1.27 1.27)
+				)
+				(justify left)
+			)
+		)
+	)
 	(global_label "BLE_P1_6"
 		(shape output)
@@
 		)
 	)
+	(global_label "SPI1_CS2"
+		(shape output)
+		(at 205.74 120.65 0)
+		(fields_autoplaced yes)
+		(effects
+			(font
+				(size 1.27 1.27)
+			)
+			(justify left)
+		)
+		(property "Intersheetrefs" "${INTERSHEET_REFS}"
+			(at 217.6756 120.65 0)
+			(show_name no)
+			(do_not_autoplace no)
+			(effects
+				(font
+					(size 1.27 1.27)
+				)
+				(justify left)
+			)
+		)
+	)
 	(global_label "BLE_P2_7"
 		(shape output)
@@
 		)
 	)
+	(global_label "I2C3_SDA"
+		(shape bidirectional)
+		(at 113.03 147.32 180)
+		(effects
+			(font
+				(size 1.27 1.27)
+			)
+			(justify right)
+		)
+		(property "Intersheetrefs" "${INTERSHEET_REFS}"
+			(at 113.03 147.32 0)
+			(show_name no)
+			(do_not_autoplace no)
+			(effects
+				(font
+					(size 1.27 1.27)
+				)
+			)
+		)
+		(property "Intersheetref" "${INTERSHEET_REFS}"
+			(at 113.03 147.32 0)
+			(hide yes)
+			(show_name no)
+			(do_not_autoplace no)
+			(effects
+				(font
+					(size 1.27 1.27)
+				)
+			)
+		)
+	)
 	(global_label "EEPROM_SDA"
 		(shape bidirectional)
@@
 	)
 	(global_label "EEPROM_SCL"
-		(shape output)
+		(shape bidirectional)
 		(at 147.32 82.55 90)
 		(effects
@@
 		)
 	)
-	(embedded_fonts no)
 )
