File: SignalProcessing.kicad_sch (KiCad schematic)
At the start: 60 parts, among them J10 Header_50mil_1x05, J5 Header_100mil_1x06, J6 Header_100mil_1x06, J9 Header_50mil_1x05, U14 AD9833BRMZ-REEL7, U15 ADS131M04IPWR, U16 AD826

Commit message: Revision B semi-final
Parts:
- J10: value Header_50mil_1x05 -> Header_50mil_1x08; footprint sldrnrd:Header_50mil_1x05 -> sldrnrd:Header_50mil_1x08; symbol sldrnrd:Connector/50Mil/Header_50mil_1x05 -> sldrnrd:Connector/50Mil/Header_50mil_1x08
Connections:
- net 3V3_Sensors: now also J10.02 (2)
- net ADC_CLOCK: now also J10.05 (5); no longer J10.02 (2)
- net ADC_CS: now also J10.04 (4)
- net ADC_MISO: now also J10.07 (7); no longer J10.04 (4)
- net ADC_MOSI: now also J10.06 (6); no longer J10.03 (3)
- net ADC_SCK: now also J10.08 (8); no longer J10.05 (5)
- new net SPI1_CS2: J10.03 (3)
Changed lines of the file:
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@@
 	(wire
 		(pts
+			(xy 208.28 251.46) (xy 195.58 251.46)
+		)
+		(stroke
+			(width 0)
+			(type default)
+		)
+	)
+	(wire
+		(pts
 			(xy 85.09 264.16) (xy 85.09 266.7)
 		)
@@
 	(wire
 		(pts
+			(xy 195.58 251.46) (xy 195.58 250.19)
+		)
+		(stroke
+			(width 0)
+			(type default)
+		)
+	)
+	(wire
+		(pts
 			(xy 69.85 83.82) (xy 60.96 83.82)
 		)
@@
 	(wire
 		(pts
+			(xy 195.58 250.19) (xy 193.04 250.19)
+		)
+		(stroke
+			(width 0)
+			(type default)
+		)
+	)
+	(wire
+		(pts
 			(xy 326.39 102.87) (xy 326.39 104.14)
 		)
@@
 	(wire
 		(pts
+			(xy 198.12 248.92) (xy 198.12 246.38)
+		)
+		(stroke
+			(width 0)
+			(type default)
+		)
+	)
+	(wire
+		(pts
 			(xy 160.02 81.28) (xy 163.83 81.28)
 		)
@@
 	(wire
 		(pts
-			(xy 205.74 251.46) (xy 205.74 265.43)
+			(xy 205.74 243.84) (xy 205.74 265.43)
 		)
 		(stroke
@@
 	(wire
 		(pts
+			(xy 208.28 243.84) (xy 205.74 243.84)
+		)
+		(stroke
+			(width 0)
+			(type default)
+		)
+	)
+	(wire
+		(pts
 			(xy 97.79 149.86) (xy 101.6 149.86)
 		)
@@
 	(wire
 		(pts
+			(xy 208.28 248.92) (xy 198.12 248.92)
+		)
+		(stroke
+			(width 0)
+			(type default)
+		)
+	)
+	(wire
+		(pts
 			(xy 280.67 102.87) (xy 280.67 104.14)
 		)
@@
 	(wire
 		(pts
-			(xy 72.39 172.72) (xy 72.39 173.99)
+			(xy 198.12 246.38) (xy 193.04 246.38)
 		)
 		(stroke
@@
 	(wire
 		(pts
-			(xy 232.41 218.44) (xy 260.35 218.44)
+			(xy 208.28 246.38) (xy 203.2 246.38)
 		)
 		(stroke
@@
 	(wire
 		(pts
-			(xy 107.95 54.61) (xy 128.27 54.61)
+			(xy 72.39 172.72) (xy 72.39 173.99)
 		)
 		(stroke
@@
 	(wire
 		(pts
-			(xy 232.41 198.12) (xy 240.03 198.12)
+			(xy 232.41 218.44) (xy 260.35 218.44)
 		)
 		(stroke
@@
 	(wire
 		(pts
-			(xy 101.6 149.86) (xy 101.6 153.67)
+			(xy 107.95 54.61) (xy 128.27 54.61)
 		)
 		(stroke
@@
 	(wire
 		(pts
-			(xy 208.28 251.46) (xy 205.74 251.46)
+			(xy 232.41 198.12) (xy 240.03 198.12)
+		)
+		(stroke
+			(width 0)
+			(type default)
+		)
+	)
+	(wire
+		(pts
+			(xy 101.6 149.86) (xy 101.6 153.67)
 		)
 		(stroke
@@
 	(wire
 		(pts
+			(xy 203.2 246.38) (xy 203.2 240.03)
+		)
+		(stroke
+			(width 0)
+			(type default)
+		)
+	)
+	(wire
+		(pts
 			(xy 194.31 208.28) (xy 191.77 208.28)
 		)
@@
 		)
 	)
+	(global_label "SPI1_CS2"
+		(shape input)
+		(at 193.04 246.38 180)
+		(fields_autoplaced yes)
+		(effects
+			(font
+				(size 1.27 1.27)
+			)
+			(justify right)
+		)
+		(property "Intersheetrefs" "${INTERSHEET_REFS}"
+			(at 181.1044 246.38 0)
+			(show_name no)
+			(do_not_autoplace no)
+			(effects
+				(font
+					(size 1.27 1.27)
+				)
+				(justify right)
+			)
+		)
+	)
 	(global_label "ExciterB_ADC"
 		(shape input)
@@
 		)
 	)
+	(global_label "ADC_CS"
+		(shape input)
+		(at 193.04 250.19 180)
+		(fields_autoplaced yes)
+		(effects
+			(font
+				(size 1.27 1.27)
+			)
+			(justify right)
+		)
+		(property "Intersheetrefs" "${INTERSHEET_REFS}"
+			(at 182.9791 250.19 0)
+			(show_name no)
+			(do_not_autoplace no)
+			(effects
+				(font
+					(size 1.27 1.27)
+				)
+				(justify right)
+			)
+		)
+	)
 	(global_label "ExciterA_ADC"
 		(shape input)
@@
 	)
 	(symbol
+		(lib_id "sldrnrd:PowerFlag/3V3")
+		(at 203.2 240.03 0)
+		(unit 1)
+		(body_style 1)
+		(exclude_from_sim no)
+		(in_bom yes)
+		(on_board yes)
+		(in_pos_files yes)
+		(dnp no)
+		(property "Reference" "#PWR0188"
+			(at 203.2 243.84 0)
+			(hide yes)
+			(show_name no)
+			(do_not_autoplace no)
+			(effects
+				(font
+					(size 1.27 1.27)
+				)
+			)
+		)
+		(property "Value" "3V3_Sensors"
+			(at 203.2 235.712 0)
+			(show_name no)
+			(do_not_autoplace no)
+			(effects
+				(font
+					(size 1.27 1.27)
+				)
+			)
+		)
+		(property "Footprint" ""
+			(at 203.2 240.03 0)
+			(hide yes)
+			(show_name no)
+			(do_not_autoplace no)
+			(effects
+				(font
+					(size 1.27 1.27)
+				)
+			)
+		)
+		(property "Datasheet" "~"
+			(at 203.2 240.03 0)
+			(hide yes)
+			(show_name no)
+			(do_not_autoplace no)
+			(effects
+				(font
+					(size 1.27 1.27)
+				)
+			)
+		)
+		(property "Description" "Power symbol creates a global label with name \"3V3\", 3.3V supply"
+			(at 203.2 240.03 0)
+			(hide yes)
+			(show_name no)
+			(do_not_autoplace no)
+			(effects
+				(font
+					(size 1.27 1.27)
+				)
+			)
+		)
+		(pin "1"
+		)
+		(instances
+			(project "Levelmeter"
+				(path "/7d35597c-fbf9-4ce7-8410-0e7922679ea3/8fba0ce8-7d88-4764-99d3-e22ea4fdebc5"
+					(reference "#PWR0188")
+					(unit 1)
+				)
+			)
+		)
+	)
+	(symbol
 		(lib_id "sldrnrd:Capacitor/C0603_220n")
 		(at 255.27 227.33 0)
@@
 	)
 	(symbol
-		(lib_id "sldrnrd:Connector/50Mil/Header_50mil_1x05")
-		(at 214.63 256.54 0)
+		(lib_id "sldrnrd:Connector/50Mil/Header_50mil_1x08")
+		(at 214.63 252.73 0)
 		(unit 1)
 		(body_style 1)
@@
 		(fields_autoplaced yes)
 		(property "Reference" "J10"
-			(at 219.71 255.2699 0)
+			(at 219.71 251.4599 0)
 			(show_name no)
 			(do_not_autoplace no)
@@
 			)
 		)
-		(property "Value" "Header_50mil_1x05"
-			(at 219.71 257.8099 0)
+		(property "Value" "Header_50mil_1x08"
+			(at 219.71 253.9999 0)
 			(show_name no)
 			(do_not_autoplace no)
@@
 			)
 		)
-		(property "Footprint" "sldrnrd:Header_50mil_1x05"
+		(property "Footprint" "sldrnrd:Header_50mil_1x08"
 			(at 214.63 267.97 0)
 			(hide yes)
@@
 			)
 		)
-		(property "Description" "1.27mm pitch pin header, single row, 5-pin, THT"
+		(property "Description" "1.27mm pitch pin header, single row, 8-pin, THT"
 			(at 214.63 273.05 0)
 			(hide yes)
@@
 		(pin "01"
 		)
+		(pin "08"
+		)
+		(pin "07"
+		)
+		(pin "06"
+		)
 		(instances
