File: connectors.kicad_sch (KiCad schematic)
At the start: 17 parts, among them J2 USB_C, J4 Header_50mil_2x07, J7 JST_PH_2.0mm_1x03

Commit message: Board layout without errors
Parts:
- renumbered C39 to C44, C41 to C45, C43 to C46, J4 to J3, J7 to J4, R27 to R29, R28 to R30, R29 to R31, R30 to R32, R31 to R33, R37 to R35
Changed lines of the file:
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@@
 		(in_pos_files yes)
 		(dnp no)
-		(property "Reference" "R28"
+		(property "Reference" "R30"
 			(at 84.582 72.39 90)
 			(show_name no)
@@
 			(project "Levelmeter"
 				(path "/7d35597c-fbf9-4ce7-8410-0e7922679ea3/7286337d-4cd5-4f95-b550-04c2e962fc51"
-					(reference "R28")
+					(reference "R30")
 					(unit 1)
 				)
@@
 		(in_pos_files yes)
 		(dnp no)
-		(property "Reference" "#PWR101"
+		(property "Reference" "#PWR0110"
 			(at 82.55 88.9 0)
 			(hide yes)
@@
 			(project "Levelmeter"
 				(path "/7d35597c-fbf9-4ce7-8410-0e7922679ea3/7286337d-4cd5-4f95-b550-04c2e962fc51"
-					(reference "#PWR101")
+					(reference "#PWR0110")
 					(unit 1)
 				)
@@
 		(in_pos_files yes)
 		(dnp no)
-		(property "Reference" "C43"
+		(property "Reference" "C46"
 			(at 347.98 66.04 90)
 			(show_name no)
@@
 			(project "Levelmeter"
 				(path "/7d35597c-fbf9-4ce7-8410-0e7922679ea3/7286337d-4cd5-4f95-b550-04c2e962fc51"
-					(reference "C43")
+					(reference "C46")
 					(unit 1)
 				)
@@
 		(dnp no)
 		(fields_autoplaced yes)
-		(property "Reference" "#PWR123"
+		(property "Reference" "#PWR0122"
 			(at 345.44 45.72 0)
 			(hide yes)
@@
 			(project "Levelmeter"
 				(path "/7d35597c-fbf9-4ce7-8410-0e7922679ea3/7286337d-4cd5-4f95-b550-04c2e962fc51"
-					(reference "#PWR123")
+					(reference "#PWR0122")
 					(unit 1)
 				)
@@
 		(in_pos_files yes)
 		(dnp no)
-		(property "Reference" "#PWR102"
+		(property "Reference" "#PWR0111"
 			(at 88.9 88.9 0)
 			(hide yes)
@@
 			(project "Levelmeter"
 				(path "/7d35597c-fbf9-4ce7-8410-0e7922679ea3/7286337d-4cd5-4f95-b550-04c2e962fc51"
-					(reference "#PWR102")
+					(reference "#PWR0111")
 					(unit 1)
 				)
@@
 		(in_pos_files yes)
 		(dnp no)
-		(property "Reference" "C41"
+		(property "Reference" "C45"
 			(at 219.71 73.66 90)
 			(show_name no)
@@
 			(project "Levelmeter"
 				(path "/7d35597c-fbf9-4ce7-8410-0e7922679ea3/7286337d-4cd5-4f95-b550-04c2e962fc51"
-					(reference "C41")
+					(reference "C45")
 					(unit 1)
 				)
@@
 		(in_pos_files yes)
 		(dnp no)
-		(property "Reference" "#PWR107"
+		(property "Reference" "#PWR0116"
 			(at 173.99 46.99 0)
 			(hide yes)
@@
 			(project "Levelmeter"
 				(path "/7d35597c-fbf9-4ce7-8410-0e7922679ea3/7286337d-4cd5-4f95-b550-04c2e962fc51"
-					(reference "#PWR107")
+					(reference "#PWR0116")
 					(unit 1)
 				)
@@
 		(in_pos_files yes)
 		(dnp no)
-		(property "Reference" "#PWR124"
+		(property "Reference" "#PWR0123"
 			(at 345.44 81.28 0)
 			(hide yes)
@@
 			(project "Levelmeter"
 				(path "/7d35597c-fbf9-4ce7-8410-0e7922679ea3/7286337d-4cd5-4f95-b550-04c2e962fc51"
-					(reference "#PWR124")
+					(reference "#PWR0123")
 					(unit 1)
 				)
@@
 		(dnp no)
 		(fields_autoplaced yes)
-		(property "Reference" "J7"
+		(property "Reference" "J4"
 			(at 365.76 52.0699 0)
 			(show_name no)
@@
 			(project "Levelmeter"
 				(path "/7d35597c-fbf9-4ce7-8410-0e7922679ea3/7286337d-4cd5-4f95-b550-04c2e962fc51"
-					(reference "J7")
+					(reference "J4")
 					(unit 1)
 				)
@@
 		(in_pos_files yes)
 		(dnp no)
-		(property "Reference" "#PWR103"
+		(property "Reference" "#PWR0112"
 			(at 93.98 88.9 0)
 			(hide yes)
@@
 			(project "Levelmeter"
 				(path "/7d35597c-fbf9-4ce7-8410-0e7922679ea3/7286337d-4cd5-4f95-b550-04c2e962fc51"
-					(reference "#PWR103")
+					(reference "#PWR0112")
 					(unit 1)
 				)
@@
 		(in_pos_files yes)
 		(dnp no)
-		(property "Reference" "R31"
+		(property "Reference" "R33"
 			(at 121.412 73.66 90)
 			(show_name no)
@@
 			(project "Levelmeter"
 				(path "/7d35597c-fbf9-4ce7-8410-0e7922679ea3/7286337d-4cd5-4f95-b550-04c2e962fc51"
-					(reference "R31")
+					(reference "R33")
 					(unit 1)
 				)
@@
 		(in_pos_files yes)
 		(dnp no)
-		(property "Reference" "#PWR95"
+		(property "Reference" "#PWR0107"
 			(at 40.64 87.63 0)
 			(hide yes)
@@
 			(project "Levelmeter"
 				(path "/7d35597c-fbf9-4ce7-8410-0e7922679ea3/7286337d-4cd5-4f95-b550-04c2e962fc51"
-					(reference "#PWR95")
+					(reference "#PWR0107")
 					(unit 1)
 				)
@@
 		(in_pos_files yes)
 		(dnp no)
-		(property "Reference" "#PWR97"
+		(property "Reference" "#PWR0109"
 			(at 48.26 87.63 0)
 			(hide yes)
@@
 			(project "Levelmeter"
 				(path "/7d35597c-fbf9-4ce7-8410-0e7922679ea3/7286337d-4cd5-4f95-b550-04c2e962fc51"
-					(reference "#PWR97")
+					(reference "#PWR0109")
 					(unit 1)
 				)
@@
 		(in_pos_files yes)
 		(dnp no)
-		(property "Reference" "R29"
+		(property "Reference" "R31"
 			(at 101.092 72.39 90)
 			(show_name no)
@@
 			(project "Levelmeter"
 				(path "/7d35597c-fbf9-4ce7-8410-0e7922679ea3/7286337d-4cd5-4f95-b550-04c2e962fc51"
-					(reference "R29")
+					(reference "R31")
 					(unit 1)
 				)
@@
 		(in_pos_files yes)
 		(dnp no)
-		(property "Reference" "R30"
+		(property "Reference" "R32"
 			(at 121.412 58.42 90)
 			(show_name no)
@@
 			(project "Levelmeter"
 				(path "/7d35597c-fbf9-4ce7-8410-0e7922679ea3/7286337d-4cd5-4f95-b550-04c2e962fc51"
-					(reference "R30")
+					(reference "R32")
 					(unit 1)
 				)
@@
 		(in_pos_files yes)
 		(dnp no)
-		(property "Reference" "C39"
+		(property "Reference" "C44"
 			(at 91.44 72.39 90)
 			(show_name no)
@@
 			(project "Levelmeter"
 				(path "/7d35597c-fbf9-4ce7-8410-0e7922679ea3/7286337d-4cd5-4f95-b550-04c2e962fc51"
-					(reference "C39")
+					(reference "C44")
 					(unit 1)
 				)
@@
 		(in_pos_files yes)
 		(dnp no)
-		(property "Reference" "#PWR106"
+		(property "Reference" "#PWR0115"
 			(at 119.38 88.9 0)
 			(hide yes)
@@
 			(project "Levelmeter"
 				(path "/7d35597c-fbf9-4ce7-8410-0e7922679ea3/7286337d-4cd5-4f95-b550-04c2e962fc51"
-					(reference "#PWR106")
+					(reference "#PWR0115")
 					(unit 1)
 				)
@@
 		(in_pos_files yes)
 		(dnp no)
-		(property "Reference" "#PWR104"
+		(property "Reference" "#PWR0113"
 			(at 99.06 88.9 0)
 			(hide yes)
@@
 			(project "Levelmeter"
 				(path "/7d35597c-fbf9-4ce7-8410-0e7922679ea3/7286337d-4cd5-4f95-b550-04c2e962fc51"
-					(reference "#PWR104")
+					(reference "#PWR0113")
 					(unit 1)
 				)
@@
 		(in_pos_files yes)
 		(dnp no)
-		(property "Reference" "#PWR125"
+		(property "Reference" "#PWR0124"
 			(at 351.79 81.28 0)
 			(hide yes)
@@
 			(project "Levelmeter"
 				(path "/7d35597c-fbf9-4ce7-8410-0e7922679ea3/7286337d-4cd5-4f95-b550-04c2e962fc51"
-					(reference "#PWR125")
+					(reference "#PWR0124")
 					(unit 1)
 				)
@@
 		(in_pos_files yes)
 		(dnp no)
-		(property "Reference" "#PWR108"
+		(property "Reference" "#PWR0117"
 			(at 173.99 85.09 0)
 			(hide yes)
@@
 			(project "Levelmeter"
 				(path "/7d35597c-fbf9-4ce7-8410-0e7922679ea3/7286337d-4cd5-4f95-b550-04c2e962fc51"
-					(reference "#PWR108")
+					(reference "#PWR0117")
 					(unit 1)
 				)
@@
 		(in_pos_files yes)
 		(dnp no)
-		(property "Reference" "#PWR116"
+		(property "Reference" "#PWR0120"
 			(at 217.17 85.09 0)
 			(hide yes)
@@
 			(project "Levelmeter"
 				(path "/7d35597c-fbf9-4ce7-8410-0e7922679ea3/7286337d-4cd5-4f95-b550-04c2e962fc51"
-					(reference "#PWR116")
+					(reference "#PWR0120")
 					(unit 1)
 				)
@@
 		(in_pos_files yes)
 		(dnp no)
-		(property "Reference" "#PWR115"
+		(property "Reference" "#PWR0119"
 			(at 217.17 46.99 0)
 			(hide yes)
@@
 			(project "Levelmeter"
 				(path "/7d35597c-fbf9-4ce7-8410-0e7922679ea3/7286337d-4cd5-4f95-b550-04c2e962fc51"
-					(reference "#PWR115")
+					(reference "#PWR0119")
 					(unit 1)
 				)
@@
 		(in_pos_files yes)
 		(dnp no)
-		(property "Reference" "#PWR117"
+		(property "Reference" "#PWR0121"
 			(at 278.13 88.9 0)
 			(hide yes)
@@
 			(project "Levelmeter"
 				(path "/7d35597c-fbf9-4ce7-8410-0e7922679ea3/7286337d-4cd5-4f95-b550-04c2e962fc51"
-					(reference "#PWR117")
+					(reference "#PWR0121")
 					(unit 1)
 				)
@@
 		(in_pos_files yes)
 		(dnp no)
-		(property "Reference" "R37"
+		(property "Reference" "R35"
 			(at 335.28 53.848 90)
 			(show_name no)
@@
 			(project "Levelmeter"
 				(path "/7d35597c-fbf9-4ce7-8410-0e7922679ea3/7286337d-4cd5-4f95-b550-04c2e962fc51"
-					(reference "R37")
+					(reference "R35")
 					(unit 1)
 				)
@@
 		(in_pos_files yes)
 		(dnp no)
-		(property "Reference" "#PWR96"
+		(property "Reference" "#PWR0108"
 			(at 44.45 43.18 0)
 			(hide yes)
@@
 			(project "Levelmeter"
 				(path "/7d35597c-fbf9-4ce7-8410-0e7922679ea3/7286337d-4cd5-4f95-b550-04c2e962fc51"
-					(reference "#PWR96")
+					(reference "#PWR0108")
 					(unit 1)
 				)
@@
 		(in_pos_files yes)
 		(dnp no)
-		(property "Reference" "J4"
+		(property "Reference" "J3"
 			(at 186.69 47.752 0)
 			(show_name no)
@@
 			(project "Levelmeter"
 				(path "/7d35597c-fbf9-4ce7-8410-0e7922679ea3/7286337d-4cd5-4f95-b550-04c2e962fc51"
-					(reference "J4")
+					(reference "J3")
 					(unit 1)
 				)
@@
 		(in_pos_files yes)
 		(dnp no)
-		(property "Reference" "#PWR111"
+		(property "Reference" "#PWR0118"
 			(at 198.12 85.09 0)
 			(hide yes)
@@
 			(project "Levelmeter"
 				(path "/7d35597c-fbf9-4ce7-8410-0e7922679ea3/7286337d-4cd5-4f95-b550-04c2e962fc51"
-					(reference "#PWR111")
+					(reference "#PWR0118")
 					(unit 1)
 				)
@@
 		(in_pos_files yes)
 		(dnp no)
-		(property "Reference" "R27"
+		(property "Reference" "R29"
 			(at 42.672 71.12 90)
 			(show_name no)
@@
 			(project "Levelmeter"
 				(path "/7d35597c-fbf9-4ce7-8410-0e7922679ea3/7286337d-4cd5-4f95-b550-04c2e962fc51"
-					(reference "R27")
+					(reference "R29")
 					(unit 1)
 				)
@@
 		(in_pos_files yes)
 		(dnp no)
-		(property "Reference" "#PWR105"
+		(property "Reference" "#PWR0114"
 			(at 119.38 43.18 0)
 			(hide yes)
@@
 			(project "Levelmeter"
 				(path "/7d35597c-fbf9-4ce7-8410-0e7922679ea3/7286337d-4cd5-4f95-b550-04c2e962fc51"
-					(reference "#PWR105")
+					(reference "#PWR0114")
 					(unit 1)
 				)

Commit message: Schematic checks, some smaller corrections, debug UART pinout corrected on programming header
Parts:
- added C71: 1n, sldrnrd:C_0603, symbol sldrnrd:Capacitor/C0603_1n
Connections:
- net DEBUG_UART_MCU_TO_PC: now also J3.14; no longer J3.02 (2)
- net DEBUG_UART_PC_TO_MCU: now also J3.13; no longer J3.01 (1)
- net GND: now also C71.2; no longer J3.13, J3.14
- net TEMP_SENSE_EXT: now also C71.1
- net 3V3 renamed 3V3_STANDBY
Other:
- moved on the sheet: C45, R34

Commit message: Revision B semi-final
Parts:
- added J12: Header_50mil_1x06, sldrnrd:Header_50mil_1x06, symbol sldrnrd:Connector/50Mil/Header_50mil_1x06
Connections:
- net GND: now also J12.01 (1)
- new net 3V3_Sensors: J12.02 (2)
- new net AUX1: J12.05 (5)
- new net AUX2: J12.06 (6)
- new net I2C3_SCL: J12.03 (3)
- new net I2C3_SDA: J12.04 (4)
Other:
- note added: "Extra I2C interface I2C3"
