File: Levelmeter.kicad_pcb (KiCad board)
At the start: 4 copper layers, 90 x 70 mm, 187 parts, among them J1 JST_PH_2.0mm_1x02, J10 Header_50mil_1x05, J11 Header_50mil_1x05, J2 USB_C, J3 Header_50mil_2x07, J4 JST_PH_2.0mm_1x03, J5 Header_100mil_1x06, J6 Header_100mil_1x06, J7 Header_100mil_1x06, J8 Header_50mil_1x03, J9 Header_50mil_1x05, Q1 AO3401A, Q2 AO3401A, Q3 FS8205A, Q4 AO3400A, Q5 AO3400A, SW1 PEC11R-4215F-S0024, SW2 PEC11R-4215F-S0024, U1 LP5907MFX-3.3/NOPB, U10 BL24C256A-SFRC, U11 BME280, U12 SN74HC14PWR, U13 TMP236A4DBZR, U14 AD9833BRMZ-REEL7, U15 ADS131M04IPWR, U16 AD826, U2 DW01A, U3 LP5907MFX-3.3/NOPB, U4 TP4056, U5 HX4002-MFC, U6 LM27761DSGR, U7 STM32G0B1RET6, U8 RN4871-I/RM128, U9 SN74AHCT244DBR, Y1 Q13FC1350000400, Y2 X50328MSB2GI

Commit message: Revision B semi-final
Parts:
- added J12: Header_50mil_1x06, sldrnrd:Header_50mil_1x06, F.Cu at (109.4, 54.6)
- J10: value Header_50mil_1x05 -> Header_50mil_1x08; footprint sldrnrd:Header_50mil_1x05 -> sldrnrd:Header_50mil_1x08
- moved R32 1.00 mm to (55.6, 89.2)
- moved R33 1.00 mm to (55.6, 87.5)
- moved J10 0.40 mm to (86.0, 41.8)
- moved D4 0.25 mm to (78.0, 60.0)
- moved R13 0.25 mm to (81.2, 60.0)
- moved C71 0.20 mm to (86.4, 61.6)
- moved R35 0.20 mm to (83.2, 61.6)
Connections:
- J10 pad 02: ADC_CLOCK -> 3V3_Sensors
- J10 pad 03: ADC_MOSI -> SPI1_CS2
- J10 pad 04: ADC_MISO -> ADC_CS
- J10 pad 05: ADC_SCK -> ADC_CLOCK
- U7 pad 13: unconnected-(U7-PC0-Pad13) -> I2C3_SCL
- U7 pad 14: unconnected-(U7-PC1-Pad14) -> I2C3_SDA
- U7 pad 42: unconnected-(U7-PA10-Pad42) -> SPI1_CS2
- U7 pad 47: unconnected-(U7-PA15-Pad47) -> AUX1
- U7 pad 48: unconnected-(U7-PC8-Pad48) -> AUX2
Routing:
- net SPI1_CS2: track 0.00 -> 46.1 mm, vias 0 -> 4
- net AUX2: track 0.00 -> 28.5 mm, vias 0 -> 2
- net AUX1: track 0.00 -> 27.6 mm, vias 0 -> 2
- net 3V3_Sensors: track 78.5 -> 100.4 mm, vias 4 -> 6
- net I2C3_SCL: track 0.00 -> 12.0 mm
- net I2C3_SDA: track 0.00 -> 10.7 mm
- net ADC_CS: track 20.7 -> 29.5 mm
- net 3V3: track 246.9 -> 240.5 mm
- net ADC_CLOCK: track 43.7 -> 41.3 mm
- net DEBUG_UART_MCU_TO_PC: track 48.1 -> 50.2 mm, vias 2 -> 4
- net ADC_SCK: track 27.0 -> 25.5 mm
- net ADC_MISO: track 26.1 -> 24.6 mm
- net DEBUG_UART_PC_TO_MCU: track 48.9 -> 50.0 mm, vias 2 -> 4
- net ADC_MOSI: track 27.6 -> 26.5 mm
- net BATTERY_SENSE: track 23.2 -> 22.7 mm
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Other:
- board text added: "I2C3"

Commit message: Levelmeter Rev B as ordered
Routing:
- net TEMP_SENSE_EXT: track 10.6 -> 11.8 mm
