File: Levelmeter_RevA/Levelmeter.kicad_pcb (KiCad board)
At the start: 4 copper layers, 90 x 70 mm, 187 parts, among them J1 JST_PH_2.0mm_1x02, J10 Header_50mil_1x05, J11 Header_50mil_1x05, J2 USB_C, J3 Header_50mil_2x07, J4 JST_PH_2.0mm_1x03, J5 Header_100mil_1x06, J6 Header_100mil_1x06, J7 Header_100mil_1x06, J8 Header_50mil_1x03, J9 Header_50mil_1x05, Q1 AO3401A, Q2 AO3401A, Q3 FS8205A, Q4 AO3400A, Q5 AO3400A, SW1 PEC11R-4215F-S0024, SW2 PEC11R-4215F-S0024, U1 LP5907MFX-3.3/NOPB, U10 BL24C256A-SFRC, U11 BME280, U12 SN74HC14PWR, U13 TMP236A4DBZR, U14 AD9833BRMZ-REEL7, U15 ADS131M04IPWR, U16 AD826, U2 DW01A, U3 LP5907MFX-3.3/NOPB, U4 TP4056, U5 HX4002-MFC, U6 LM27761DSGR, U7 STM32G0B1RET6, U8 RN4871-I/RM128, U9 SN74AHCT244DBR, Y1 Q13FC1350000400, Y2 X50328MSB2GI

Commit message: Levelmeter REV B started
Parts:
- moved C42 14.7 mm to (77.5, 70.0), turned to 180 degrees
- moved U13 10.7 mm to (77.0, 67.2), turned to 0 degrees
- moved R28 9.66 mm to (83.6, 66.2)
- moved C72 9.61 mm to (86.0, 67.0)
- moved C71 1.17 mm to (85.4, 62.4)
- moved R35 1.13 mm to (82.4, 62.6)
- moved R59 0.20 mm to (89.0, 55.8)
Connections:
- U7 pad 15: CHARGE_SENSE -> unconnected-(U7-PC2-Pad15)
- U7 pad 20: BATTERY_SENSE -> CHARGE_SENSE
- U7 pad 31: TEMP_SENSE_EXT -> LED_STATUS
- U7 pad 32: TEMP_SENSE -> LED_PWR
- U7 pad 33: LED_PWR -> unconnected-(U7-PB13-Pad33)
- U7 pad 34: LED_STATUS -> unconnected-(U7-PB14-Pad34)
- U7 pad 42: unconnected-(U7-PA10-Pad42) -> TEMP_SENSE_EXT
- U7 pad 47: unconnected-(U7-PA15-Pad47) -> BATTERY_SENSE
- U7 pad 48: unconnected-(U7-PC8-Pad48) -> TEMP_SENSE
Routing:
- net Net-(U13-VOUT): track 19.3 -> 4.63 mm
- net BATTERY_SENSE: track 23.2 -> 10.9 mm, vias 2 -> 0
- net 5V0: track 298.4 -> 289.8 mm, vias 10 -> 12
- net LED_STATUS: track 7.66 -> 11.8 mm
- net TEMP_SENSE_EXT: track 10.6 -> 6.53 mm, vias 2 -> 0
- net Net-(J4-Pad3): track 44.7 -> 42.3 mm
- net LED_PWR: track 8.33 -> 10.3 mm
- net CHARGE_SENSE: track 52.2 -> 50.5 mm, vias 4 -> 2
- net TEMP_SENSE: track 6.52 -> 4.92 mm
- net DEBUG_UART_PC_TO_MCU: track 48.9 -> 49.7 mm
- net DEBUG_UART_MCU_TO_PC: track 48.1 -> 48.8 mm
- net 3V3: track 246.9 -> 247.5 mm
- net GND: vias 339 -> 337
Other:
- board text added: "soldernerd.com LEVELMETER 2026 - Rev A"
- board text removed: "Status"
- board text removed: "soldernerd.com LEVELMETER 2026 - Rev B"
