File: Levelmeter_RevA/mcu.kicad_sch (KiCad schematic)
At the start: 15 parts, among them J8 Header_50mil_1x03, U7 STM32G0B1RET6, U8 RN4871-I/RM128, Y1 Q13FC1350000400, Y2 X50328MSB2GI

Commit message: Levelmeter REV B started
Connections:
- net BATTERY_SENSE: now also U7.47 (PA15); no longer U7.20 (PA3)
- net CHARGE_SENSE: now also U7.20 (PA3); no longer U7.15 (PC2)
- net LED_PWR: now also U7.32 (PB12); no longer U7.33 (PB13)
- net LED_STATUS: now also U7.31 (PB11); no longer U7.34 (PB14)
- net TEMP_SENSE: now also U7.48 (PC8); no longer U7.32 (PB12)
- net TEMP_SENSE_EXT: now also U7.42 (PA10); no longer U7.31 (PB11)
Changed lines of the file:
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@@
 	(wire
 		(pts
-			(xy 113.03 151.13) (xy 120.65 151.13)
-		)
-		(stroke
-			(width 0)
-			(type default)
-		)
-	)
-	(wire
-		(pts
 			(xy 116.84 97.79) (xy 120.65 97.79)
 		)
@@
 	(wire
 		(pts
+			(xy 200.66 97.79) (xy 205.74 97.79)
+		)
+		(stroke
+			(width 0)
+			(type default)
+		)
+	)
+	(wire
+		(pts
 			(xy 298.45 172.72) (xy 298.45 180.34)
 		)
@@
 	(wire
 		(pts
+			(xy 200.66 120.65) (xy 205.74 120.65)
+		)
+		(stroke
+			(width 0)
+			(type default)
+		)
+	)
+	(wire
+		(pts
 			(xy 331.47 118.11) (xy 340.36 118.11)
 		)
@@
 	(wire
 		(pts
-			(xy 200.66 151.13) (xy 205.74 151.13)
-		)
-		(stroke
-			(width 0)
-			(type default)
-		)
-	)
-	(wire
-		(pts
 			(xy 91.44 116.84) (xy 97.79 116.84)
 		)
@@
 	(wire
 		(pts
-			(xy 200.66 154.94) (xy 205.74 154.94)
+			(xy 143.51 166.37) (xy 143.51 172.72)
 		)
 		(stroke
@@
 	(wire
 		(pts
+			(xy 200.66 101.6) (xy 205.74 101.6)
+		)
+		(stroke
+			(width 0)
+			(type default)
+		)
+	)
+	(wire
+		(pts
 			(xy 361.95 129.54) (xy 361.95 154.94)
 		)
@@
 	(wire
 		(pts
-			(xy 143.51 166.37) (xy 143.51 172.72)
-		)
-		(stroke
-			(width 0)
-			(type default)
-		)
-	)
-	(wire
-		(pts
 			(xy 154.94 82.55) (xy 154.94 86.36)
 		)
@@
 	(global_label "TEMP_SENSE"
 		(shape input)
-		(at 189.23 172.72 270)
+		(at 205.74 97.79 0)
 		(effects
 			(font
 				(size 1.27 1.27)
 			)
-			(justify right)
+			(justify left)
 		)
 		(property "Intersheetrefs" "${INTERSHEET_REFS}"
-			(at 189.23 172.72 90)
+			(at 205.74 97.79 0)
 			(show_name no)
 			(do_not_autoplace no)
@@
 		)
 		(property "Intersheetref" "${INTERSHEET_REFS}"
-			(at 189.23 172.72 90)
+			(at 205.74 97.79 0)
 			(hide yes)
 			(show_name no)
@@
 	(global_label "CHARGE_SENSE"
 		(shape input)
-		(at 113.03 151.13 180)
+		(at 143.51 172.72 270)
 		(fields_autoplaced yes)
 		(effects
@@
 		)
 		(property "Intersheetrefs" "${INTERSHEET_REFS}"
-			(at 95.6516 151.13 0)
+			(at 143.51 190.0984 90)
 			(show_name no)
 			(do_not_autoplace no)
@@
 	(global_label "BATTERY_SENSE"
 		(shape input)
-		(at 143.51 172.72 270)
+		(at 205.74 101.6 0)
 		(fields_autoplaced yes)
 		(effects
@@
 				(size 1.27 1.27)
 			)
-			(justify right)
+			(justify left)
 		)
 		(property "Intersheetrefs" "${INTERSHEET_REFS}"
-			(at 143.51 190.5217 90)
+			(at 223.5417 101.6 0)
 			(show_name no)
 			(do_not_autoplace no)
@@
 					(size 1.27 1.27)
 				)
-				(justify right)
+				(justify left)
 			)
 		)
@@
 	(global_label "LED_STATUS"
 		(shape output)
-		(at 205.74 151.13 0)
+		(at 185.42 172.72 270)
 		(effects
 			(font
 				(size 1.27 1.27)
 			)
-			(justify left)
+			(justify right)
 		)
 		(property "Intersheetrefs" "${INTERSHEET_REFS}"
-			(at 205.74 151.13 0)
+			(at 185.42 172.72 90)
 			(show_name no)
 			(do_not_autoplace no)
@@
 		)
 		(property "Intersheetref" "${INTERSHEET_REFS}"
-			(at 205.74 151.13 0)
+			(at 185.42 172.72 90)
 			(hide yes)
 			(show_name no)
@@
 	(global_label "TEMP_SENSE_EXT"
 		(shape input)
-		(at 185.42 172.72 270)
+		(at 205.74 120.65 0)
 		(effects
 			(font
 				(size 1.27 1.27)
 			)
-			(justify right)
+			(justify left)
 		)
 		(property "Intersheetrefs" "${INTERSHEET_REFS}"
-			(at 185.42 172.72 90)
+			(at 205.74 120.65 0)
 			(show_name no)
 			(do_not_autoplace no)
@@
 		)
 		(property "Intersheetref" "${INTERSHEET_REFS}"
-			(at 185.42 172.72 90)
+			(at 205.74 120.65 0)
 			(hide yes)
 			(show_name no)
@@
 	(global_label "LED_PWR"
 		(shape output)
-		(at 205.74 154.94 0)
+		(at 189.23 172.72 270)
 		(effects
 			(font
 				(size 1.27 1.27)
 			)
-			(justify left)
+			(justify right)
 		)
 		(property "Intersheetrefs" "${INTERSHEET_REFS}"
-			(at 205.74 154.94 0)
+			(at 189.23 172.72 90)
 			(show_name no)
 			(do_not_autoplace no)
@@
 		)
 		(property "Intersheetref" "${INTERSHEET_REFS}"
-			(at 205.74 154.94 0)
+			(at 189.23 172.72 90)
 			(hide yes)
 			(show_name no)
@@
 		)
 	)
-	(embedded_fonts no)
 )
