File: Levelmeter_RevA/power.kicad_sch (KiCad schematic)
At the start: 45 parts, among them J11 Header_50mil_1x05, J7 Header_100mil_1x06, SW1 PEC11R-4215F-S0024, SW2 PEC11R-4215F-S0024, U10 BL24C256A-SFRC, U11 BME280, U12 SN74HC14PWR, U13 TMP236A4DBZR, U9 SN74AHCT244DBR

Commit message: Levelmeter REV B started
Parts:
- removed BZ1: CPT-9019S-SMT-TR, sldrnrd:CPT-9019S, symbol sldrnrd:Audio/CPT-9019S-SMT-TR
- removed C30, C31, C37, C39: 10n, sldrnrd:C_0603, symbol sldrnrd:Capacitor/C0603_10n
- removed C32, C33, C34, C36, C38, C40, C41, C42, C43: 100n, sldrnrd:C_0603, symbol sldrnrd:Capacitor/C0603_100n
- removed C35: 2u2, sldrnrd:C_0805, symbol sldrnrd:Capacitor/C0805_2u2
- removed C72: 1n, sldrnrd:C_0603, symbol sldrnrd:Capacitor/C0603_1n
- removed D3, D4: LED_Red_0603, sldrnrd:LED_0603, symbol sldrnrd:LED/LED_Red_0603
- removed DS1: LS027B7DH01, sldrnrd:Display_LS027B7DH01, symbol sldrnrd:Display/LS027B7DH01
- removed J11: Header_50mil_1x05, sldrnrd:Header_50mil_1x05, symbol sldrnrd:Connector/50Mil/Header_50mil_1x05
- removed J7: Header_100mil_1x06, sldrnrd:Header_100mil_1x06, symbol sldrnrd:Connector/100Mil/Header_100mil_1x06
- removed R12, R13: 1k, sldrnrd:R_0603, symbol sldrnrd:Resistor/R0603_1k
- removed R14, R15, R16, R17, R18, R19, R22, R23, R24, R25, R26, R27: 33k, sldrnrd:R_0603, symbol sldrnrd:Resistor/R0603_33k
- removed R20, R21: 5k1, sldrnrd:R_0603, symbol sldrnrd:Resistor/R0603_5k1
- removed R28: 2k, sldrnrd:R_0603, symbol sldrnrd:Resistor/R0603_2k
- removed SW1, SW2: PEC11R-4215F-S0024, sldrnrd:RotaryEncoder_PEC11R, symbol sldrnrd:InputDevice/RotaryEncoder/PEC11R-4215F-S0024
- removed U10: BL24C256A-SFRC, sldrnrd:TSSOP-8, symbol sldrnrd:Memory/EEPROM/BL24C256A-SFRC
- removed U11: BME280, sldrnrd:LGA-8_2.5x2.5mm_P0.65mm, symbol sldrnrd:Sensor/BME280
- removed U12: SN74HC14PWR, sldrnrd:TSSOP-14, symbol sldrnrd:Logic/74/SN74HC14PWR
- removed U13: TMP236A4DBZR, sldrnrd:SOT-23-3, symbol sldrnrd:Sensor/TMP236A4DBZR
- removed U9: SN74AHCT244DBR, sldrnrd:SSOP-20, symbol sldrnrd:Logic/74/SN74AHCT244DBR
- added C1, C15, C4: 1u, sldrnrd:C_0805, symbol sldrnrd:Capacitor/C0805_1u
- added C10, C12, C18, C19, C2, C21, C5, C6: 100n, sldrnrd:C_0603, symbol sldrnrd:Capacitor/C0603_100n
- added C11, C13, C16, C17, C20, C3, C69, C7, C70, C8, C9: 10u, sldrnrd:C_0805, symbol sldrnrd:Capacitor/C0805_10u
- added C14: 2u2, sldrnrd:C_0805, symbol sldrnrd:Capacitor/C0805_2u2
- added D1, D2: LED_Red_0603, sldrnrd:LED_0603, symbol sldrnrd:LED/LED_Red_0603
- added J1: JST_PH_2.0mm_1x02, sldrnrd:JST_PH_2.0mm_1x02, symbol sldrnrd:Connector/JST/JST_PH_2.0mm_1x02
- added Q1, Q2: AO3401A, sldrnrd:SOT-23-3, symbol sldrnrd:Transistor/MosfetP/AO3401A
- added Q3: FS8205A, sldrnrd:SOT-23-6, symbol sldrnrd:Transistor/MosfetN/FS8205A_TechPublic
- added Q4, Q5: AO3400A, sldrnrd:SOT-23-3, symbol sldrnrd:Transistor/MosfetN/AO3400A
- added R1, R10, R57: 100k, sldrnrd:R_0603, symbol sldrnrd:Resistor/R0603_100k
- added R11, R5: 33k, sldrnrd:R_0603, symbol sldrnrd:Resistor/R0603_33k
- added R2, R6, R7: 1k, sldrnrd:R_0603, symbol sldrnrd:Resistor/R0603_1k
- added R3: 470R, sldrnrd:R_0603, symbol sldrnrd:Resistor/R0603_470R
- added R4: 2k, sldrnrd:R_0603, symbol sldrnrd:Resistor/R0603_2k
- added R8: 180k, sldrnrd:R_0603, symbol sldrnrd:Resistor/R0603_180k
- added R9: 68k, sldrnrd:R_0603, symbol sldrnrd:Resistor/R0603_68k
- added U1, U3: LP5907MFX-3.3/NOPB, sldrnrd:SOT-23-5, symbol sldrnrd:Power/LinearRegulator/LP5907MFX-3.3_NOPB
- added U2: DW01A, sldrnrd:SOT-23-6, symbol sldrnrd:Power/BatteryManagement/DW01A_PUOLOP
- added U4: TP4056, sldrnrd:ESOP-8, symbol sldrnrd:Power/BatteryManagement/TP4056
- added U5: HX4002-MFC, sldrnrd:SOT-23-6, symbol sldrnrd:Power/ChargePump/HX4002-MFC
- added U6: LM27761DSGR, sldrnrd:WSON-8-2x2-EP, symbol sldrnrd:Power/ChargePump/LM27761DSGR
Connections:
- net 3V3: now also D1.2 (A), D2.2 (A), Q2.3 (D), Q5.1 (G), R57.1, U3.3 (EN)
- net 3V3_STANDBY: now also C2.1, C3.1, C69.1, C70.1, Q2.2 (S), U1.5 (OUT)
- net 5V0: now also C10.1, C17.1, C18.1, C8.1, U5.1 (VOUT), U6.1 (VIN), U6.6 (EN)
- net GND: now also C1.2, C10.2, C11.2, C12.2, C13.2, C16.2, C17.2, C18.2, C19.2, C2.2, C20.2, C21.2, C3.2, C4.2, C6.2, C69.2, C7.2, C70.2, C8.2, C9.2, Q3.3 (S2), Q4.2 (S), Q5.2 (S), R2.2, R4.1, R57.2, R9.2, U1.2 (GND), U3.2 (GND), U4.1 (TEMP), U4.3 (GND), U4.9 (EP), U5.2 (GND), U6.2 (GND), U6.9 (EP)
- new net: D1.1 (K), R6.1
- new net: Q3.4 (G2), U2.3 (OC)
- new net: Q3.6 (G1), U2.1 (OD)
- new net: R8.2, R9.1, U6.5 (VFB)
- new net: Q4.3 (D), R5.2, U4.8 (CE)
- new net: C5.1, R3.1, U2.5 (VCC)
- new net: Q5.3 (D), R11.2
- new net: C14.1, U5.6 (C+)
- new net: C14.2, U5.4 (C-)
- new net: D2.1 (K), R7.1
- new net: C16.1, U6.3 (CPOUT)
- new net: Q1.1 (G), R1.2
- new net: C15.1, U6.8 (C1+)
- new net: C15.2, U6.7 (C1-)
- new net: R2.1, U2.2 (VM)
- new net: R4.2, U4.2 (PROG)
- new net  ~{3v3_EN}: Q2.1 (G)
- new net -4V5: C20.1, C21.1, R8.1, U6.4 (VOUT)
- new net 3V3_Sensors: C6.1, C7.1, U3.5 (OUT)
- new net 5V_EN: U5.3 (EN)
- new net BAT+: J1.1, Q1.3 (D)
- new net BAT-: C5.2, J1.2, Q3.1 (S1), R1.1, U2.6 (GND)
- new net BATTERY_SENSE: C19.1, R10.2, R11.1
- new net CHARGE_SENSE: R6.2, U4.7 (~{CHRG})
- new net STANDBY_SENSE: R7.2, U4.6 (~{STDBY})
- new net VCC: C1.1, C11.1, C12.1, C13.1, C4.1, Q1.2 (S), R10.1, R3.2, U1.1 (IN), U1.3 (EN), U3.1 (IN), U4.5 (BAT), U5.5 (VIN)
- new net V_USB: C9.1, R5.1, U4.4 (VCC)
- new net ~{CHARGE_EN}: Q4.1 (G)
- no-connect marks 0 -> 3
Other:
- note added: "Cell Protection (DW01A + FS8205A)"
- note added: "LM27761 Voltage Inverter"
- note added: "LP5907MFX-3.3 LDO"
- note added: "LP5907MFX-3.3 LDO for sensors"
- note added: "Reverse Polarity Protection"
- note added: "SD6210A 5V Charge Pump"
- note added: "TP4056 LiPo Charger"
- note added: "VBAT Monitoring (ADC)"
- note removed: "24LC256 EEPROM"
- note removed: "Encoder 1"
- note removed: "Encoder 2"
- note removed: "Encoder Debouncing"
- note removed: "Environmental sensor BME280"
- note removed: "J4 — FH12-10S-0.5SH (Display FPC)"
- note removed: "LM35 Temperature Sensor"
- note removed: "Piezo Buzzer (BZ1)"
- note removed: "SN74AHCT244 Level Shifter (3.3V to 5V)"
- note removed: "Status LEDs"
- title: User Interface & Peripherals -> Power Supply
